File: deflection_amp_3/power_supply.kicad_sch (KiCad schematic)
At the start: 40 parts, among them U1 AP2205-ADJ, U2 AP2205-ADJ, U3 LT8365, U4 LT8365

Commit message: fixed BOM + DAC footprint
Parts:
- C10, C9: JLCPCB P/N FS43X105K251EGG -> 0805F224M500NT
- C13, C14, C15: JLCPCB P/N FS55X105K251EGG -> FS43X105K251EGG
Changed lines of the file:
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@@
 			)
 		)
-		(property "JLCPCB P/N" "FS43X105K251EGG"
+		(property "JLCPCB P/N" "0805F224M500NT"
 			(at 114.3 123.19 0)
 			(effects
@@
 			)
 		)
-		(property "JLCPCB P/N" "FS55X105K251EGG"
+		(property "JLCPCB P/N" "FS43X105K251EGG"
 			(at 189.23 91.44 0)
 			(effects
@@
 			)
 		)
-		(property "JLCPCB P/N" "FS43X105K251EGG"
+		(property "JLCPCB P/N" "0805F224M500NT"
 			(at 114.3 67.31 0)
 			(effects
@@
 			)
 		)
-		(property "JLCPCB P/N" "FS55X105K251EGG"
+		(property "JLCPCB P/N" "FS43X105K251EGG"
 			(at 189.23 35.56 0)
 			(effects
@@
 			)
 		)
-		(property "JLCPCB P/N" "FS55X105K251EGG"
+		(property "JLCPCB P/N" "FS43X105K251EGG"
 			(at 158.75 85.09 0)
 			(effects
