File: deflection_amp_3/deflection_amp_3.kicad_pcb (KiCad board)
At the start: 2 copper layers, 100 x 86 mm, 202 parts, among them J1 USB_C_Receptacle_USB2.0_14P, J2 POWER INPUT, J3 OFFSET REFERENCE, J4 DEFLECTION OUT, Q1 FMMT458TA, Q10 FMMT558TA, Q11 FMMT458TA, Q12 FMMT558TA, Q13 FMMT558TA, Q14 FMMT458TA, Q15 FMMT558TA, Q16 FMMT458TA, Q17 FMMT458TA, Q18 FMMT558TA, Q19 FMMT458TA, Q2 FMMT558TA, Q20 FMMT558TA, Q21 FMMT558TA, Q22 FMMT458TA, Q23 FMMT558TA, Q24 FMMT458TA, Q25 FMMT458TA, Q26 FMMT558TA, Q27 FMMT458TA, Q28 FMMT558TA, Q29 FMMT558TA, Q3 FMMT458TA, Q30 FMMT458TA, Q31 FMMT558TA, Q32 FMMT458TA, Q4 FMMT558TA, Q5 FMMT558TA, Q6 FMMT458TA, Q7 FMMT558TA, Q8 FMMT458TA, Q9 FMMT458TA, SW1 RESET, SW2 PROG, U1 AP2205-ADJ, U10 LMH6639, U11 LMH6639, U12 LMH6639, U2 AP2205-ADJ, U3 LT8365, U4 LT8365, U5 W25Q128JVS, U6 RP2040, U7 MCP4822, U8 MCP4822, U9 LMH6639, Y1 ABM8-272-T3

Commit message: fixed BOM + DAC footprint
Parts:
- U7, U8: footprint Package_SO:SOIC-8_5.3x5.3mm_P1.27mm -> MCP4822-E_SN:SOIC127P599X175-8N
Routing:
- net LDAC2: track 18.3 -> 24.1 mm
- net LDAC1: track 34.6 -> 31.8 mm
- net +3.3V: track 204.9 -> 207.1 mm
- net SPI1_MOSI: track 15.0 -> 13.7 mm
- net SPI0_MOSI: track 29.9 -> 28.8 mm
- net /High Voltage Amp - Y1/INPUT: track 21.2 -> 22.1 mm
- net /High Voltage Amp - X2/INPUT: track 17.5 -> 18.4 mm
- net /High Voltage Amp - X1/INPUT: track 34.4 -> 35.3 mm
- net /High Voltage Amp - Y2/INPUT: track 33.2 -> 34.1 mm
- net SPI1_CS: track 18.5 -> 18.0 mm
- net GND: vias 23 -> 24

Commit message: cleanup
Parts:
- J1: footprint Connector_USB:USB_C_Receptacle_JAE_DX07S016JA1R1500 -> Connector_USB:USB_C_Receptacle_Palconn_UTC16-G
- moved J1 0.55 mm to (141.6, 111.0)
Routing:
- net /RP2040 + DACs/USB+: track 5.35 -> 7.40 mm
