File: deflection_amp_3/deflection_amp_3.kicad_sch (KiCad schematic)
At the start: 14 parts, among them J1 USB_C_Receptacle_USB2.0_14P, J2 POWER INPUT, J3 OFFSET REFERENCE, J4 DEFLECTION OUT

Commit message: cleanup
Parts:
- F1: JLCPCB P/N MFU0805FF02000P100 -> MFU0805FF02000P500
- J1: footprint Connector_USB:USB_C_Receptacle_JAE_DX07S016JA1R1500 -> Connector_USB:USB_C_Receptacle_Palconn_UTC16-G; JLCPCB P/N DX07S016JA1R1500 -> TYPE-C 16PIN 2MD(073)
Changed lines of the file:
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@@
 			)
 		)
-		(property "Footprint" "Connector_USB:USB_C_Receptacle_JAE_DX07S016JA1R1500"
+		(property "Footprint" "Connector_USB:USB_C_Receptacle_Palconn_UTC16-G"
 			(at 34.29 78.74 0)
 			(effects
@@
 			)
 		)
-		(property "JLCPCB P/N" "DX07S016JA1R1500"
+		(property "JLCPCB P/N" "TYPE-C 16PIN 2MD(073)"
 			(at 30.48 58.42 0)
 			(effects
@@
 			)
 		)
-		(property "JLCPCB P/N" "MFU0805FF02000P100"
+		(property "JLCPCB P/N" "MFU0805FF02000P500"
 			(at 38.1 36.83 0)
 			(effects
