File: deflection_amp_3/main_amp.kicad_sch (KiCad schematic)
At the start: 26 parts, among them Q1 FMMT458TA, Q2 FMMT558TA, Q3 FMMT458TA, Q4 FMMT558TA, Q5 FMMT558TA, Q6 FMMT458TA, Q7 FMMT558TA, Q8 FMMT458TA, U9 LMH6639

Commit message: cleanup
Parts:
- Q2, Q4, Q5, Q7: JLCPCB P/N FMMT558QTA -> FMMT560QTA
Changed lines of the file:
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@@
 			)
 		)
-		(property "JLCPCB P/N" "FMMT558QTA"
+		(property "JLCPCB P/N" "FMMT560QTA"
 			(at 147.32 62.23 0)
 			(effects
@@
 			)
 		)
-		(property "JLCPCB P/N" "FMMT558QTA"
+		(property "JLCPCB P/N" "FMMT560QTA"
 			(at 142.24 100.33 0)
 			(effects
@@
 			)
 		)
-		(property "JLCPCB P/N" "FMMT558QTA"
+		(property "JLCPCB P/N" "FMMT560QTA"
 			(at 129.54 100.33 0)
 			(effects
@@
 			)
 		)
-		(property "JLCPCB P/N" "FMMT558QTA"
+		(property "JLCPCB P/N" "FMMT560QTA"
 			(at 160.02 62.23 0)
 			(effects
