File: main_supply_3_revised/main_supply_3_revised/filament.kicad_sch (KiCad schematic)
At the start: 37 parts, among them Q3 NMOS, T3 YA9033-ALD, U4 PC817, U5 LM5155DSSR, U6 TL431DBZ

Commit message: defl 5 + mainboard 3
Parts:
- removed D17: D, Diode_SMD:D_SMA, symbol Device:D
- added C48: C, Capacitor_SMD:C_0603_1608Metric, symbol Device:C
- added D25: D_Schottky, Diode_SMD:D_SMA, symbol Device:D_Schottky
- added D26, D27: D_Schottky, Diode_SMD:D_SOD-123, symbol Device:D_Schottky
- added D28: Generic_Triac_A1A2G, Package_TO_SOT_SMD:SOT-223, symbol Triac_Thyristor:Generic_Triac_A1A2G
- added D30: LED, LED_SMD:LED_0603_1608Metric, symbol Device:LED
- added F2: 2A, Fuse:Fuseholder_Littelfuse_Nano2_154x, symbol Device:Fuse
- added R44: R_US, Resistor_SMD:R_0603_1608Metric, symbol Device:R_US
- added R46: 220, Resistor_SMD:R_0603_1608Metric, symbol Device:R_US
- added R52: 33k, Resistor_SMD:R_0603_1608Metric, symbol Device:R_US
- added R58: 20k, Resistor_SMD:R_0603_1608Metric, symbol Device:R_US
- added R60: 3.9k, Resistor_SMD:R_0603_1608Metric, symbol Device:R_Small_US
- added U6: TL431DBZ, Package_TO_SOT_SMD:SOT-23, symbol Reference_Voltage:TL431DBZ
- Q3: value NMOS -> Si7450DP; footprint Package_TO_SOT_SMD:TO-252-3_TabPin4 -> Package_SO:PowerPAK_SO-8_Single
- R45: renamed from R49; value 50k -> 10k
- R59: value 20k -> 21k
- RV3: renamed from RV5; footprint Potentiometer_THT:Potentiometer_Bourns_3296W_Vertical -> Potentiometer_THT:Potentiometer_Bourns_3296Y_Vertical
- renumbered C30 to C40, C31 to C41, C32 to C42, C33 to C43, C34 to C44, C57 to C45, C35 to C46, C36 to C47, C38 to C49, C39 to C50, C37 to C51, C41 to C52, C40 to C53, D18 to D29, R47 to R42, R48 to R43, R50 to R47, R51 to R48, R53 to R49, R52 to R50, R56 to R51, R54 to R53, R58 to R54, R57 to R56, R60 to R57, RS3 to RS4, U6 to U7
Connections:
- net +12V_IN: now also R60.1
- net CATHODE: now also D29.1 (K), C48.2, D28.1 (A1), R58.2, U6.3 (A)
- net FILAMENT: now also R54.1, D28.2 (A2), F2.2, R46.1, R52.1; no longer C41.1, C42.1, C43.1, C44.1, R47.1, R48.1
- net GND: now also D30.1 (K)
- net MOS_DRAIN_FIL: now also Q3.5 (D); no longer Q3.1 (D)
- net MOS_SOURCE_FIL: now also Q3.1 (S), Q3.2 (S)
- net VCC_FIL: no longer R54.1
- net at C51.1, R53.2, U4.2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: now also D27.2 (A)
- net at R49.2: now also Q3.4 (G); no longer Q3.2 (G)
- net at T3.7, T3.8: now also D25.2 (A)
- net GATE_FIL: no longer names the net of R49.1, U5.3 (GATE)
- net PGOOD_FIL: no longer names the net of U5.11 (PGOOD)
- net PGOOD_FIL: no longer D29.1 (K)
- new net: C48.1, D26.2 (A), D27.1 (K), R44.2
- new net: R52.2, R58.1, U6.2 (REF)
- new net: D30.2 (A), R60.2
- new net TRIAC_GATE: D28.3 (G), R46.2, U6.1 (K)
- new net UNFUSED_FILAMENT: C41.1, C42.1, C43.1, C44.1, D25.1 (K), D26.1 (K), F2.1, R44.1, R47.1, R48.1
- no-connect marks 0 -> 1
Other:
- note added: "5.71V - 6.42V Voltage Adjust"
- note added: "6.625V cutoff"
- note added: "ISO BARRIER"
- note added: "over-voltage crowbar"
- note added: "secondary side soft-start"
- moved on the sheet: C40, C41, C42, C43, C44, C45, C46, C47, C49, C50, C51, C52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
