File: main_supply_3_revised/main_supply_3_revised/hv_minus.kicad_sch (KiCad schematic)
At the start: 53 parts, among them Q1 NMOS, U1 LM5155DSSR, U2 TLV237

Commit message: defl 5 + mainboard 3
Parts:
- removed C15: 100p, Capacitor_SMD:C_0603_1608Metric, symbol Device:C
- removed C4, C6, C8: 220n, Capacitor_SMD:C_2220_5750Metric, symbol Device:C_Small
- removed C7, C9: 100n, Capacitor_SMD:C_1812_4532Metric, symbol Device:C_Small
- removed D2, D3, D5, D6, D7: D, Diode_SMD:D_SMA, symbol Device:D
- removed Q1: NMOS, Package_TO_SOT_SMD:TO-252-3_TabPin4, symbol Simulation_SPICE:NMOS
- removed R13, R14, R16, R17, R18, R19, R20, R21, R22: 1Meg, Resistor_SMD:R_1206_3216Metric, symbol Device:R_US
- removed R5, R6, R9: 20, Resistor_SMD:R_1206_3216Metric, symbol Device:R_Small_US
- removed RV1: 1Meg, Potentiometer_THT:Potentiometer_Bourns_3296W_Vertical, symbol Device:R_Potentiometer_US
- added C20, C21, C22, C23, C24, C26, C27, C28, C29, C30, C55: 100n, Capacitor_SMD:C_1812_4532Metric, symbol Device:C_Small
- added C54: 20p, Capacitor_SMD:C_0603_1608Metric, symbol Device:C
- added D13, D14, D15, D16, D17, D18, D19, D20, D21, D22, D31: D, Diode_SMD:D_SMA, symbol Device:D
- added Q2: Si7450DP, Package_SO:PowerPAK_SO-8_Single, symbol Simulation_SPICE:NMOS
- added R29, R30, R31, R32, R33, R34, R35, R36, R37, R38: 1Meg, Resistor_SMD:R_1206_3216Metric, symbol Device:R_US
- added T2: DA2032-AL, DA2032-AL:DA2032-AL, symbol DA2032-AL:DA2032-AL
- C25: renamed from C1; footprint Capacitor_SMD:C_0603_1608Metric -> Capacitor_SMD:C_0805_2012Metric
- R23: renamed from R3; value 50k -> 10k
- R24: renamed from R4; footprint Resistor_SMD:R_0603_1608Metric -> Resistor_SMD:R_1206_3216Metric
- R25: renamed from R15; value 470 -> 4.7k
- RV2: value 4.7k -> 20k; footprint Potentiometer_THT:Potentiometer_Bourns_3296W_Vertical -> Potentiometer_THT:Potentiometer_Bourns_3296Y_Vertical
- renumbered C2 to C31, C3 to C32, C5 to C33, C58 to C34, C10 to C35, C11 to C36, C12 to C37, C13 to C38, C14 to C39, D1 to D23, D8 to D24, NT1 to NT2, R1 to R21, R2 to R22, R7 to R26, R8 to R27, R10 to R28, R11 to R39, R23 to R40, R12 to R41, RS1 to RS2, U1 to U2, U2 to U3
Connections:
- net +12V_IN: now also T2.3, T2.4, T2.5, T2.6
- net CS: now also Q2.1 (S), Q2.2 (S), Q2.3 (S)
- net FB_HV: now also C54.1
- net FB_HV_LADDER: now also C54.2, R29.1
- net GND: now also D24.1 (K), C26.2, D13.1 (K), T2.1
- net MOS_DRAIN: now also Q2.5 (D), T2.10, T2.7, T2.8, T2.9
- net PGOOD_HV: now also D24.2 (A), R28.2; no longer D24.1 (K)
- net at R26.2: now also Q2.4 (G)
- new net: C20.1, C21.2, D13.2 (A), D14.1 (K)
- new net: C26.1, C27.2, D14.2 (A), D15.1 (K)
- new net: R34.2, R35.1
- new net: R35.2, R36.1
- new net: C29.1, C30.2, D20.2 (A), D21.1 (K)
- new net: C28.1, C29.2, D18.2 (A), D19.1 (K)
- new net: R36.2, R37.1
- new net: R29.2, R30.1
- new net: R30.2, R31.1
- new net: R31.2, R32.1
- new net: C27.1, C28.2, D16.2 (A), D17.1 (K)
- new net: R37.2, R38.1
- new net: C24.1, C55.2, D21.2 (A), D22.1 (K)
- new net: C23.1, C24.2, D19.2 (A), D20.1 (K)
- new net: C21.1, C22.2, D15.2 (A), D16.1 (K)
- new net: C22.1, C23.2, D17.2 (A), D18.1 (K)
- new net: C30.1, D22.2 (A), D31.1 (K)
- new net: R33.2, R34.1
- new net: R32.2, R33.1
- new net -HV: C55.1, D31.2 (A), R38.2
- new net HV_SEC: C20.2, T2.12
Other:
- note added: "10 Meg 2KV rated 200V per 1206"
- note added: "400-2000V voltage adj."
- note added: "fix this shit"
- note added: "see about changing the 100n caps for 10n ?"
- note removed: "10 Meg"
- note removed: "2KV"
- note removed: "check if this is too much?"
- note removed: "is D8/R4 necessary?"
- note removed: "set max current sense"
- note removed: "what are these caps even rated for?"
- moved on the sheet: C25, C34, C36, D24, R24, R25, R28, R40, RV2, U3
