File: main_supply_3_revised/main_supply_3_revised/hv_pos.kicad_sch (KiCad schematic)
At the start: 49 parts, among them Q2 NMOS, U3 LM5155DSSR

Commit message: defl 5 + mainboard 3
Parts:
- removed C16: 100n, Capacitor_SMD:C_1812_4532Metric, symbol Device:C_Small
- removed C17, C19, C23: 220n, Capacitor_SMD:C_2220_5750Metric, symbol Device:C_Small
- removed D11: D, Diode_SMD:D_SMA, symbol Device:D
- removed R24, R25, R28: 20, Resistor_SMD:R_1206_3216Metric, symbol Device:R_Small_US
- added C10, C11, C2, C3, C4, C5, C7, C8, C9: 100n, Capacitor_SMD:C_1812_4532Metric, symbol Device:C_Small
- added D3, D4, D5, D6, D7, D8: D, Diode_SMD:D_SMA, symbol Device:D
- added T1: DA2032-AL, DA2032-AL:DA2032-AL, symbol DA2032-AL:DA2032-AL
- C6: renamed from C20; footprint Capacitor_SMD:C_0603_1608Metric -> Capacitor_SMD:C_0805_2012Metric
- Q1: renamed from Q2; value NMOS -> Si7450DP; footprint Package_TO_SOT_SMD:TO-252-2 -> Package_SO:PowerPAK_SO-8_Single
- R4: renamed from R30; footprint Resistor_SMD:R_0603_1608Metric -> Resistor_SMD:R_1206_3216Metric
- RV1: renamed from RV3; footprint Potentiometer_THT:Potentiometer_Bourns_3296W_Vertical -> Potentiometer_THT:Potentiometer_Bourns_3296Y_Vertical
- renumbered C18 to C1, C21 to C12, C22 to C13, C24 to C14, C25 to C15, C26 to C16, C27 to C17, C28 to C18, C29 to C19, D13 to D1, D14 to D11, D16 to D12, D12 to D2, NT2 to NT1, R26 to R1, R44 to R10, R43 to R11, R42 to R12, R41 to R13, R40 to R14, R39 to R15, R38 to R16, R37 to R17, R35 to R18, R34 to R19, R27 to R2, R36 to R20, R29 to R3, R31 to R5, R32 to R6, R33 to R7, R46 to R8, R45 to R9, RS2 to RS1, U3 to U1
Connections:
- net +12V_IN: now also T1.3, T1.4, T1.5, T1.6
- net +PDA: now also D10.1 (K), R18.2, C11.1; no longer R18.1
- net CS: now also Q1.1 (S), Q1.2 (S)
- net FB_PDA: now also R8.2, RV1.1; no longer R9.1, RV1.3
- net GND: now also D1.2 (A), D12.1 (K), C7.2, T1.12
- net MOS_DRAIN: now also Q1.5 (D), T1.10, T1.7, T1.8, T1.9; no longer Q1.2 (D)
- net PGOOD_HV: now also D12.2 (A), R7.2; no longer D12.1 (K)
- net at D10.2 (A): now also D9.1 (K), C5.1
- net at R13.2: now also R14.1; no longer R14.2
- net at D1.1 (K): now also C1.1, D2.2 (A), C2.2
- net at D2.1 (K): now also C7.1, C8.2, D3.2 (A); no longer C1.2
- net at R16.1: now also R15.2; no longer R17.2
- net at R16.2: now also R17.1; no longer R15.1
- net at D9.2 (A): now also C10.1, C11.2, D8.1 (K); no longer D10.1 (K)
- net at R5.2: now also Q1.4 (G); no longer Q1.1 (G)
- new net: C8.1, C9.2, D4.1 (K), D5.2 (A)
- new net: C2.1, C3.2, D3.1 (K), D4.2 (A)
- new net: C4.1, C5.2, D7.1 (K), D8.2 (A)
- new net: C10.2, C9.1, D6.1 (K), D7.2 (A)
- new net: R9.1, RV1.3
- new net: R17.2, R18.1
- new net: C3.1, C4.2, D5.1 (K), D6.2 (A)
- new net: R14.2, R15.1
- new net PDA_SEC: C1.2, T1.1
Other:
- note added: "10 Meg 2KV rated 200V per 1206"
- note added: "400-2000V voltage adj."
- note added: "see about changing the 100n caps for 10n ?"
- note removed: "10 Meg"
- note removed: "2KV"
- note removed: "400-2KV"
- moved on the sheet: C1, C12, C13, C14, C15, C16, C17, C18, C19, C6, D1, D11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
