File: main_supply_3_revised/main_supply_3_revised/main_supply_3_revised.kicad_pcb (KiCad board)
At the start: 2 copper layers, 100 x 100 mm, 147 parts, among them J1 Conn_01x02_Pin, J2 A3_EN, J3 A3, J5 A2_EN, J6 FIL_EN, Q1 NMOS, Q2 NMOS, Q3 NMOS, T3 YA9033-ALD, U1 LM5155DSSR, U2 TLV237, U3 LM5155DSSR, U4 PC817, U5 LM5155DSSR, U6 TL431DBZ

Commit message: defl 5 + mainboard 3
Parts:
- removed C57: 1u, Capacitor_SMD:C_0603_1608Metric
- removed C58: 100n, Capacitor_SMD:C_0603_1608Metric
- removed J2: A3_EN, Connector_PinHeader_2.54mm:PinHeader_1x02_P2.54mm_Vertical
- removed the R10 at (105.3, 101.8)
- removed the R11 at (115.8, 101.8)
- removed the R12 at (122.6, 105.5)
- removed the R13 at (186.6, 78.0)
- removed the R14 at (181.3, 78.0)
- removed the R15 at (107.8, 83.1)
- removed the R16 at (175.9, 78.0)
- removed the R17 at (170.7, 78.0)
- removed the R18 at (165.5, 78.0)
- removed the R9 at (186.4, 94.5)
- removed RS3: 0.02, Resistor_SMD:R_1206_3216Metric
- removed RV5: 4.7k, Potentiometer_THT:Potentiometer_Bourns_3296W_Vertical
- added C42: 10u, Capacitor_SMD:C_0805_2012Metric, F.Cu at (142.6, 135.8)
- added C43: 10u, Capacitor_SMD:C_0805_2012Metric, F.Cu at (146.5, 135.8)
- added C44: 100u, Capacitor_SMD:CP_Elec_6.3x7.7, F.Cu at (152.9, 133.1)
- added C45: 1u, Capacitor_SMD:C_0603_1608Metric, F.Cu at (116.8, 145.5)
- added C46: 10u, Capacitor_SMD:C_0805_2012Metric, F.Cu at (120.5, 128.9)
- added C47: 10u, Capacitor_SMD:C_0805_2012Metric, F.Cu at (123.5, 128.9)
- added C48: C, Capacitor_SMD:C_0603_1608Metric, F.Cu at (155.1, 147.9)
- added C49: 470p, Capacitor_SMD:C_0603_1608Metric, F.Cu at (110.9, 135.5)
- added C50: 1u, Capacitor_SMD:C_0603_1608Metric, F.Cu at (116.8, 143.8)
- added C51: 220n, Capacitor_SMD:C_0603_1608Metric, F.Cu at (148.4, 142.3)
- added C52: 47n, Capacitor_SMD:C_0603_1608Metric, F.Cu at (107.6, 138.6)
- added C53: 220n, Capacitor_SMD:C_0603_1608Metric, F.Cu at (119.0, 148.1)
- added C54: 20p, Capacitor_SMD:C_0603_1608Metric, F.Cu at (107.8, 109.9)
- added C55: 100n, Capacitor_SMD:C_1812_4532Metric, F.Cu at (188.4, 114.6)
- added D15: D, Diode_SMD:D_SMA, F.Cu at (158.1, 106.9)
- added D19: D, Diode_SMD:D_SMA, F.Cu at (174.4, 106.8)
- added D20: D, Diode_SMD:D_SMA, F.Cu at (178.4, 106.8)
- added D21: D, Diode_SMD:D_SMA, F.Cu at (182.4, 106.8)
- added D22: D, Diode_SMD:D_SMA, F.Cu at (186.4, 106.7)
- added D23: LED, LED_SMD:LED_0603_1608Metric, F.Cu at (163.5, 90.0)
- added D24: LED, LED_SMD:LED_0603_1608Metric, F.Cu at (170.5, 90.0)
- added D25: D_Schottky, Diode_SMD:D_SMA, F.Cu at (141.9, 130.0)
- added D26: D_Schottky, Diode_SMD:D_SOD-123, F.Cu at (150.8, 145.5)
- added D27: D_Schottky, Diode_SMD:D_SOD-123, F.Cu at (155.9, 145.5)
- added D28: Generic_Triac_A1A2G, Package_TO_SOT_SMD:SOT-223, F.Cu at (172.0, 130.9)
- added D29: LED, LED_SMD:LED_0603_1608Metric, F.Cu at (184.5, 90.0)
- added D30: LED, LED_SMD:LED_0603_1608Metric, F.Cu at (177.5, 90.0)
- added D31: D, Diode_SMD:D_SMA, F.Cu at (190.5, 106.7)
- added D4: D, Diode_SMD:D_SMA, F.Cu at (162.1, 73.4)
- added F2: 2A, Fuse:Fuseholder_Littelfuse_Nano2_154x, F.Cu at (162.4, 132.9)
- added J4: HV OUT, Connector_JST:JST_VH_B5P-VH-B_1x05_P3.96mm_Vertical, F.Cu at (194.3, 76.6)
- added J7: FIL_EN, Connector_PinHeader_2.54mm:PinHeader_1x02_P2.54mm_Vertical, F.Cu at (102.6, 126.2)
- added R35: 1Meg, Resistor_SMD:R_1206_3216Metric, F.Cu at (168.4, 122.8)
- added R37: 1Meg, Resistor_SMD:R_1206_3216Metric, F.Cu at (178.7, 122.8)
- added R38: 1Meg, Resistor_SMD:R_1206_3216Metric, F.Cu at (183.7, 122.8)
- added R39: 2k, Resistor_SMD:R_0603_1608Metric, F.Cu at (111.6, 113.1)
- added R40: 4.7k, Resistor_SMD:R_0603_1608Metric, F.Cu at (105.1, 115.6)
- added R41: 220k, Resistor_SMD:R_0603_1608Metric, F.Cu at (105.1, 119.2)
- added R42: 50k, Resistor_SMD:R_0603_1608Metric, F.Cu at (107.5, 142.0)
- added R43: 100, Resistor_SMD:R_0603_1608Metric, F.Cu at (123.3, 134.3)
- added R44: R_US, Resistor_SMD:R_0603_1608Metric, F.Cu at (151.5, 147.9)
- added R45: 10k, Resistor_SMD:R_0603_1608Metric, F.Cu at (107.6, 143.8)
- added RS4: 0.02, Resistor_SMD:R_1206_3216Metric, F.Cu at (117.3, 134.0)
- added U7: TL431DBZ, Package_TO_SOT_SMD:SOT-23, F.Cu at (144.1, 141.9)
- C1, C20, C27, C30: value 220p -> 100n; footprint Capacitor_SMD:C_0603_1608Metric -> Capacitor_SMD:C_1812_4532Metric
- C10: value 470p -> 100n; footprint Capacitor_SMD:C_0603_1608Metric -> Capacitor_SMD:C_1812_4532Metric
- C11, C26: value 1u -> 100n; footprint Capacitor_SMD:C_0603_1608Metric -> Capacitor_SMD:C_1812_4532Metric
- C12: value 220p -> 10u; footprint Capacitor_SMD:C_0603_1608Metric -> Capacitor_SMD:C_0805_2012Metric
- C13: value 47n -> 10u; footprint Capacitor_SMD:C_0603_1608Metric -> Capacitor_SMD:C_0805_2012Metric
- C14: value 220n -> 100n
- C15: value 100p -> 470p
- C16: value 100n -> 1u; footprint Capacitor_SMD:C_1812_4532Metric -> Capacitor_SMD:C_0603_1608Metric
- C17: value 220n -> 220p; footprint Capacitor_SMD:C_2220_5750Metric -> Capacitor_SMD:C_0603_1608Metric
- C18: value 100n -> 47n; footprint Capacitor_SMD:C_1812_4532Metric -> Capacitor_SMD:C_0603_1608Metric
- C19: value 220n -> 22n; footprint Capacitor_SMD:C_2220_5750Metric -> Capacitor_SMD:C_0603_1608Metric
- C2, C21, C22, C3: value 10u -> 100n; footprint Capacitor_SMD:C_0805_2012Metric -> Capacitor_SMD:C_1812_4532Metric
- C23, C4, C8: value 220n -> 100n; footprint Capacitor_SMD:C_2220_5750Metric -> Capacitor_SMD:C_1812_4532Metric
- C24, C5: footprint Capacitor_SMD:C_0603_1608Metric -> Capacitor_SMD:C_1812_4532Metric
- C25: value 470p -> 220p; footprint Capacitor_SMD:C_0603_1608Metric -> Capacitor_SMD:C_0805_2012Metric
- C28: value 47n -> 100n; footprint Capacitor_SMD:C_0603_1608Metric -> Capacitor_SMD:C_1812_4532Metric
- C29: value 22n -> 100n; footprint Capacitor_SMD:C_0603_1608Metric -> Capacitor_SMD:C_1812_4532Metric
- C31: value 100n -> 10u; footprint Capacitor_SMD:C_0603_1608Metric -> Capacitor_SMD:C_0805_2012Metric
- C33: value 10u -> 100n; footprint Capacitor_SMD:C_0805_2012Metric -> Capacitor_SMD:C_0603_1608Metric
- C34: value 100u -> 100n; footprint Capacitor_SMD:CP_Elec_6.3x7.7 -> Capacitor_SMD:C_0603_1608Metric
- C35: value 10u -> 470p; footprint Capacitor_SMD:C_0805_2012Metric -> Capacitor_SMD:C_0603_1608Metric
- C36: value 10u -> 1u; footprint Capacitor_SMD:C_0805_2012Metric -> Capacitor_SMD:C_0603_1608Metric
- C37, C40: value 220n -> 220p
- C38: value 470p -> 47n
- C39: value 1u -> 220n
- C41: value 47n -> 100n
- C6: value 220n -> 220p; footprint Capacitor_SMD:C_2220_5750Metric -> Capacitor_SMD:C_0805_2012Metric
- D1, D14, D16, D18, D8: value LED -> D; footprint LED_SMD:LED_0603_1608Metric -> Diode_SMD:D_SMA
- D11, D12: value D -> LED; footprint Diode_SMD:D_SMA -> LED_SMD:LED_0603_1608Metric
- F1: footprint Fuse:Fuse_0805_2012Metric -> Fuse:Fuseholder_Littelfuse_Nano2_154x
- J3: value A3 -> A3_EN; footprint Connector_PinHeader_2.54mm:PinHeader_1x01_P2.54mm_Vertical -> Connector_PinHeader_2.54mm:PinHeader_1x02_P2.54mm_Vertical
- J6: value FIL_EN -> FILAMENT; footprint Connector_PinHeader_2.54mm:PinHeader_1x02_P2.54mm_Vertical -> Connector_JST:JST_VH_B2P-VH-B_1x02_P3.96mm_Vertical
- Q1, Q3: value NMOS -> Si7450DP; footprint Package_TO_SOT_SMD:TO-252-3_TabPin4 -> Package_SO:PowerPAK_SO-8_Single
- Q2: value NMOS -> Si7450DP; footprint Package_TO_SOT_SMD:TO-252-2 -> Package_SO:PowerPAK_SO-8_Single
- R19: value 1Meg -> 22k; footprint Resistor_SMD:R_1206_3216Metric -> Resistor_SMD:R_0603_1608Metric
- R20: value 1Meg -> 220k; footprint Resistor_SMD:R_1206_3216Metric -> Resistor_SMD:R_0603_1608Metric
- R21: value 1Meg -> 3.9k; footprint Resistor_SMD:R_1206_3216Metric -> Resistor_SMD:R_0603_1608Metric
- R22: value 1Meg -> 50k; footprint Resistor_SMD:R_1206_3216Metric -> Resistor_SMD:R_0603_1608Metric
- R23: value 4.7k -> 10k
- R24: value 20 -> 100
- R25: value 20 -> 4.7k; footprint Resistor_SMD:R_1206_3216Metric -> Resistor_SMD:R_0603_1608Metric
- R26: value 3.9k -> 0
- R27: value 50k -> 20
- R28: value 20 -> 2k; footprint Resistor_SMD:R_1206_3216Metric -> Resistor_SMD:R_0603_1608Metric
- R29: value 10k -> 1Meg; footprint Resistor_SMD:R_0603_1608Metric -> Resistor_SMD:R_1206_3216Metric
- R3: value 50k -> 10k
- R30: value 100 -> 1Meg; footprint Resistor_SMD:R_0603_1608Metric -> Resistor_SMD:R_1206_3216Metric
- R31: value 0 -> 1Meg; footprint Resistor_SMD:R_0603_1608Metric -> Resistor_SMD:R_1206_3216Metric
- R32: value 20 -> 1Meg; footprint Resistor_SMD:R_0603_1608Metric -> Resistor_SMD:R_1206_3216Metric
- R33: value 2k -> 1Meg; footprint Resistor_SMD:R_0603_1608Metric -> Resistor_SMD:R_1206_3216Metric
- R34: value 22k -> 1Meg; footprint Resistor_SMD:R_0603_1608Metric -> Resistor_SMD:R_1206_3216Metric
- R36: value 220k -> 1Meg; footprint Resistor_SMD:R_0603_1608Metric -> Resistor_SMD:R_1206_3216Metric
- R4: footprint Resistor_SMD:R_0603_1608Metric -> Resistor_SMD:R_1206_3216Metric
- R46: value 4.7k -> 220
- R47: value 50k -> 1k
- R48: value 100 -> 33k
- R49: value 50k -> 0
- R5: value 20 -> 0; footprint Resistor_SMD:R_1206_3216Metric -> Resistor_SMD:R_0603_1608Metric
- R50: value 1k -> 5k
- R51: value 33k -> 20
- R52: value 5k -> 33k
- R53: value 0 -> 1k
- R54: value 1k -> 2k
- R56: value 20 -> 1k
- R57: value 1k -> 50k
- R58: value 2k -> 20k
- R59: value 20k -> 21k
- R6: footprint Resistor_SMD:R_1206_3216Metric -> Resistor_SMD:R_0603_1608Metric
- R60: value 50k -> 3.9k
- R7: value 0 -> 2k
- R8: value 20 -> 4.7k
- RV1: value 1Meg -> 20k; footprint Potentiometer_THT:Potentiometer_Bourns_3296W_Vertical -> Potentiometer_THT:Potentiometer_Bourns_3296Y_Vertical
- RV2: value 4.7k -> 20k; footprint Potentiometer_THT:Potentiometer_Bourns_3296W_Vertical -> Potentiometer_THT:Potentiometer_Bourns_3296Y_Vertical
- RV3: value 20k -> 4.7k; footprint Potentiometer_THT:Potentiometer_Bourns_3296W_Vertical -> Potentiometer_THT:Potentiometer_Bourns_3296Y_Vertical
- T1, T2: value ~ -> DA2032-AL; footprint coilcraft:NA5920-AL -> DA2032-AL:DA2032-AL
- U2: value TLV237 -> LM5155DSSR; footprint Package_TO_SOT_SMD:SOT-23-5 -> LM5155:IC_LM5155DSSR
- U3: value LM5155DSSR -> TLV237; footprint LM5155:IC_LM5155DSSR -> Package_TO_SOT_SMD:SOT-23-5
- moved RV3 97.7 mm to (169.8, 145.2), turned to 0 degrees
- moved J6 94.1 mm to (195.2, 128.8), turned to -90 degrees
- moved J3 93.8 mm to (102.4, 76.8)
- moved R46 89.9 mm to (179.9, 129.2), turned to 90 degrees
- moved RV1 89.5 mm to (108.2, 67.2), turned to 0 degrees
- moved R58 80.1 mm to (183.7, 133.0), turned to -90 degrees
- moved D8 79.2 mm to (178.2, 73.4), turned to 90 degrees
- moved C22 76.4 mm to (163.8, 114.7), turned to 180 degrees
- moved C17 75.0 mm to (109.2, 76.1), turned to 180 degrees
- moved C21 73.4 mm to (155.7, 114.7), turned to 180 degrees
- moved C24 72.7 mm to (180.4, 114.6), turned to 180 degrees
- moved R24 72.3 mm to (122.0, 105.7), turned to -90 degrees
- moved R25 70.6 mm to (107.8, 106.2), turned to 180 degrees
- moved R33 68.0 mm to (158.3, 122.8)
- moved R34 67.8 mm to (163.4, 122.8)
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- renumbered R44 to R10, R43 to R11, R42 to R12, R41 to R13, R40 to R14, R39 to R15, R38 to R16, R37 to R17, R35 to R18, R45 to R9
Connections:
- C1 pad 1: /A2 Supply/+12V_IN -> Net-(D1-K)
- C1 pad 2: Net-(C1-Pad2) -> /A3 Supply/PDA_SEC
- C10 pad 1: /A2 Supply/CS_FILT -> Net-(D8-K)
- C10 pad 2: GND -> Net-(D6-K)
- C11 pad 1: /A2 Supply/VCC -> /A3 Supply/+PDA
- C11 pad 2: GND -> Net-(D8-K)
- C12 pad 1: Net-(U1-COMP) -> /A3 Supply/+12V_IN
- C12 pad 2: AGND -> GND
- C13 pad 1: Net-(U1-SS) -> /A3 Supply/+12V_IN
- C13 pad 2: AGND -> GND
- C14 pad 1: Net-(C14-Pad1) -> /A3 Supply/+12V_IN
- C14 pad 2: AGND -> GND
- C15 pad 1: /A2 Supply/FB_HV -> /A3 Supply/CS_FILT
- C15 pad 2: /A2 Supply/FB_HV_LADDER -> GND
- C16 pad 1: Net-(D11-A) -> /A3 Supply/VCC
- C16 pad 2: Net-(D10-K) -> GND
- C17 pad 1: Net-(D10-A) -> Net-(U1-COMP)
- C17 pad 2: /A3 Supply/+PDA -> AGND3
- C18 pad 1: Net-(D13-A) -> Net-(U1-SS)
- C18 pad 2: Net-(D11-A) -> AGND3
- C19 pad 1: Net-(D12-A) -> Net-(C19-Pad1)
- C19 pad 2: Net-(D10-A) -> AGND3
- C2 pad 1: /A2 Supply/+12V_IN -> Net-(D3-K)
- C2 pad 2: GND -> Net-(D1-K)
- C20 pad 1: /A3 Supply/+12V_IN -> Net-(D13-A)
- C20 pad 2: Net-(C20-Pad2) -> /A2 Supply/HV_SEC
- C21 pad 1: /A3 Supply/+12V_IN -> Net-(D15-A)
- C21 pad 2: GND -> Net-(D13-A)
- C22 pad 1: /A3 Supply/+12V_IN -> Net-(D17-A)
- C22 pad 2: GND -> Net-(D15-A)
- C23 pad 1: GND -> Net-(D19-A)
- C23 pad 2: Net-(D12-A) -> Net-(D17-A)
- C24 pad 1: /A3 Supply/+12V_IN -> Net-(D21-A)
- C24 pad 2: GND -> Net-(D19-A)
- C25 pad 1: /A3 Supply/CS_FILT -> /A2 Supply/+12V_IN
- C25 pad 2: GND -> Net-(C25-Pad2)
- C26 pad 1: /A3 Supply/VCC -> Net-(D14-A)
- C27 pad 1: Net-(U3-COMP) -> Net-(D16-A)
- C27 pad 2: AGND3 -> Net-(D14-A)
- C28 pad 1: Net-(U3-SS) -> Net-(D18-A)
- C28 pad 2: AGND3 -> Net-(D16-A)
- C29 pad 1: Net-(C29-Pad1) -> Net-(D20-A)
- C29 pad 2: AGND3 -> Net-(D18-A)
- C3 pad 1: /A2 Supply/+12V_IN -> Net-(D5-K)
- C3 pad 2: GND -> Net-(D3-K)
- C30 pad 1: /Filament Supply/+12V_IN -> Net-(D22-A)
- C30 pad 2: Net-(C30-Pad2) -> Net-(D20-A)
- C31 pad 1: /Filament Supply/FILAMENT -> /A2 Supply/+12V_IN
- C31 pad 2: /Filament Supply/CATHODE -> GND
- C32 pad 1: /Filament Supply/FILAMENT -> /A2 Supply/+12V_IN
- C32 pad 2: /Filament Supply/CATHODE -> GND
- C33 pad 1: /Filament Supply/FILAMENT -> /A2 Supply/+12V_IN
- C33 pad 2: /Filament Supply/CATHODE -> GND
- C34 pad 1: /Filament Supply/FILAMENT -> /A2 Supply/VCC
- C34 pad 2: /Filament Supply/CATHODE -> GND
- C35 pad 1: /Filament Supply/+12V_IN -> /A2 Supply/CS_FILT
- C36 pad 1: /Filament Supply/+12V_IN -> /A2 Supply/VCC
- C37 pad 1: Net-(U6-K) -> Net-(U2-COMP)
- C37 pad 2: Net-(C37-Pad2) -> AGND
- C38 pad 1: /Filament Supply/CS_FIL -> Net-(U2-SS)
- C38 pad 2: GND -> AGND
- C39 pad 1: /Filament Supply/VCC_FIL -> Net-(C39-Pad1)
- C39 pad 2: GND -> AGND
- C4 pad 1: GND -> Net-(D7-K)
- C4 pad 2: Net-(D3-K) -> Net-(D5-K)
- C40 pad 1: Net-(C40-Pad1) -> /Filament Supply/+12V_IN
- C40 pad 2: GND -> Net-(C40-Pad2)
- C41 pad 1: Net-(U5-SS) -> /Filament Supply/UNFUSED_FILAMENT
- C41 pad 2: AGND2 -> /Filament Supply/CATHODE
- C5 pad 1: /A2 Supply/+12V_IN -> Net-(D10-A)
- C5 pad 2: GND -> Net-(D7-K)
- C6 pad 1: Net-(D3-K) -> /A3 Supply/+12V_IN
- C6 pad 2: Net-(D6-K) -> Net-(C6-Pad2)
- C7 pad 2: Net-(D3-A) -> GND
- C8 pad 1: Net-(D6-K) -> Net-(D4-K)
- C8 pad 2: /A2 Supply/-2KV -> Net-(D2-K)
- C9 pad 1: Net-(D3-A) -> Net-(D6-K)
- C9 pad 2: Net-(D6-A) -> Net-(D4-K)
- D1 pad 1: GND -> Net-(D1-K)
- D1 pad 2: Net-(D1-A) -> GND
- D10 pad 1: Net-(D10-K) -> /A3 Supply/+PDA
- D11 pad 1: Net-(D11-K) -> GND
- D12 pad 1: Net-(D11-A) -> GND
- D12 pad 2: Net-(D12-A) -> /A3 Supply/PGOOD_HV
- D13 pad 1: Net-(D13-K) -> GND
- D14 pad 1: GND -> Net-(D13-A)
- D16 pad 1: /A3 Supply/PGOOD_HV -> Net-(D15-A)
- D17 pad 1: /Filament Supply/FILAMENT -> Net-(D16-A)
- D18 pad 1: /Filament Supply/PGOOD_FIL -> Net-(D17-A)
- D2 pad 2: Net-(D2-A) -> Net-(D1-K)
- D3 pad 2: Net-(D3-A) -> Net-(D2-K)
- D5 pad 1: Net-(D3-A) -> Net-(D5-K)
- D5 pad 2: Net-(D5-A) -> Net-(D4-K)
- D6 pad 2: Net-(D6-A) -> Net-(D5-K)
- D7 pad 1: Net-(D6-A) -> Net-(D7-K)
- D7 pad 2: Net-(D7-A) -> Net-(D6-K)
- D8 pad 1: /A2 Supply/PGOOD_HV -> Net-(D8-K)
- D8 pad 2: Net-(D8-A) -> Net-(D7-K)
- D9 pad 1: Net-(D9-K) -> Net-(D10-A)
- D9 pad 2: Net-(D10-K) -> Net-(D8-K)
- J3 pad 1: /A3 Supply/+PDA -> +12V
- J6 pad 1: +12V -> /Filament Supply/FILAMENT
- J6 pad 2: /Filament Supply/+12V_IN -> /Filament Supply/CATHODE
- NT1 pad 1: AGND -> AGND3
- NT2 pad 1: AGND3 -> AGND
- Q1 pad 1: /A2 Supply/MOS_DRAIN -> /A3 Supply/CS
- Q1 pad 2: Net-(Q1-G) -> /A3 Supply/CS
- Q1 pad 3: /A2 Supply/CS -> /A3 Supply/CS
- Q1 pad 4: (no net) -> Net-(Q1-G)
- Q2 pad 1: Net-(Q2-G) -> /A2 Supply/CS
- Q2 pad 2: /A3 Supply/MOS_DRAIN -> /A2 Supply/CS
- Q2 pad 3: /A3 Supply/CS -> /A2 Supply/CS
- Q3 pad 1: /Filament Supply/MOS_DRAIN_FIL -> /Filament Supply/MOS_SOURCE_FIL
- Q3 pad 2: Net-(Q3-G) -> /Filament Supply/MOS_SOURCE_FIL
- Q3 pad 4: (no net) -> Net-(Q3-G)
- R1 pad 1: /A2 Supply/+12V_IN -> /A3 Supply/+12V_IN
- R1 pad 2: Net-(D1-A) -> Net-(D11-A)
- R13 pad 2: Net-(R40-Pad2) -> Net-(R13-Pad2)
- R14 pad 1: Net-(R39-Pad2) -> Net-(R13-Pad2)
- R14 pad 2: Net-(R40-Pad2) -> Net-(R14-Pad2)
- R15 pad 1: Net-(R38-Pad2) -> Net-(R14-Pad2)
- R15 pad 2: Net-(R39-Pad2) -> Net-(R15-Pad2)
- R16 pad 1: Net-(R37-Pad2) -> Net-(R15-Pad2)
- R16 pad 2: Net-(R38-Pad2) -> Net-(R16-Pad2)
- R17 pad 1: Net-(R35-Pad2) -> Net-(R16-Pad2)
- R17 pad 2: Net-(R37-Pad2) -> Net-(R17-Pad2)
- R18 pad 1: /A3 Supply/+PDA -> Net-(R17-Pad2)
- R18 pad 2: Net-(R35-Pad2) -> /A3 Supply/+PDA
- R19 pad 1: Net-(R19-Pad1) -> Net-(U1-COMP)
- R19 pad 2: Net-(R18-Pad1) -> Net-(C19-Pad1)
- R2 pad 1: /A2 Supply/+12V_IN -> /A3 Supply/+12V_IN
- R2 pad 2: /A2 Supply/UVLO -> /A3 Supply/UVLO
- R20 pad 1: Net-(R20-Pad1) -> Net-(U1-RT)
- R20 pad 2: Net-(R19-Pad1) -> AGND3
- R21 pad 1: Net-(R21-Pad1) -> /A2 Supply/+12V_IN
- R21 pad 2: Net-(R20-Pad1) -> Net-(D23-A)
- R22 pad 1: /A2 Supply/FB_HV_LADDER -> /A2 Supply/+12V_IN
- R22 pad 2: Net-(R21-Pad1) -> /A2 Supply/UVLO
- R23 pad 1: /A2 Supply/FB_HV -> /A2 Supply/UVLO
- R24 pad 1: Net-(D9-K) -> Net-(C25-Pad2)
- R24 pad 2: /A3 Supply/+PDA -> /A2 Supply/MOS_DRAIN
- R25 pad 1: Net-(D11-K) -> /A2 Supply/FB_HV
- R25 pad 2: Net-(D10-A) -> Net-(R25-Pad2)
- R26 pad 1: /A3 Supply/+12V_IN -> Net-(U2-GATE)
- R26 pad 2: Net-(D14-A) -> Net-(Q2-G)
- R27 pad 1: /A3 Supply/+12V_IN -> /A2 Supply/CS_FILT
- R27 pad 2: /A3 Supply/UVLO -> /A2 Supply/CS
- R28 pad 1: Net-(D13-K) -> /A2 Supply/VCC
- R28 pad 2: Net-(D12-A) -> /A2 Supply/PGOOD_HV
- R29 pad 1: /A3 Supply/UVLO -> /A2 Supply/FB_HV_LADDER
- R29 pad 2: GND -> Net-(R29-Pad2)
- R3 pad 1: /A2 Supply/UVLO -> /A3 Supply/UVLO
- R30 pad 1: Net-(C20-Pad2) -> Net-(R29-Pad2)
- R30 pad 2: /A3 Supply/MOS_DRAIN -> Net-(R30-Pad2)
- R31 pad 1: Net-(U3-GATE) -> Net-(R30-Pad2)
- R31 pad 2: Net-(Q2-G) -> Net-(R31-Pad2)
- R32 pad 1: /A3 Supply/CS_FILT -> Net-(R31-Pad2)
- R32 pad 2: /A3 Supply/CS -> Net-(R32-Pad2)
- R33 pad 1: /A3 Supply/VCC -> Net-(R32-Pad2)
- R33 pad 2: Net-(D16-A) -> Net-(R33-Pad2)
- R34 pad 1: Net-(U3-COMP) -> Net-(R33-Pad2)
- R34 pad 2: Net-(C29-Pad1) -> Net-(R34-Pad2)
- R36 pad 1: Net-(U3-RT) -> Net-(R35-Pad2)
- R36 pad 2: AGND3 -> Net-(R36-Pad2)
- R4 pad 1: Net-(C1-Pad2) -> Net-(C6-Pad2)
- R4 pad 2: /A2 Supply/MOS_DRAIN -> /A3 Supply/MOS_DRAIN
- R46 pad 1: GND -> /Filament Supply/FILAMENT
- R46 pad 2: Net-(R46-Pad2) -> /Filament Supply/TRIAC_GATE
- R47 pad 1: /Filament Supply/+12V_IN -> /Filament Supply/UNFUSED_FILAMENT
- R47 pad 2: /Filament Supply/UVLO -> Net-(R47-Pad2)
- R48 pad 1: Net-(C30-Pad2) -> /Filament Supply/UNFUSED_FILAMENT
- R48 pad 2: /Filament Supply/MOS_DRAIN_FIL -> Net-(U7-REF)
- R49 pad 1: /Filament Supply/UVLO -> Net-(U5-GATE)
- R49 pad 2: GND -> Net-(Q3-G)
- R5 pad 1: Net-(D2-A) -> Net-(U1-GATE)
- R5 pad 2: Net-(D3-K) -> Net-(Q1-G)
- R50 pad 1: /Filament Supply/FILAMENT -> /Filament Supply/VCC_FIL
- R50 pad 2: Net-(R50-Pad2) -> /Filament Supply/COMP_FB_FIL
- R51 pad 1: /Filament Supply/FILAMENT -> /Filament Supply/CS_FIL
- R51 pad 2: Net-(U6-REF) -> /Filament Supply/MOS_SOURCE_FIL
- R52 pad 1: /Filament Supply/VCC_FIL -> /Filament Supply/FILAMENT
- R52 pad 2: /Filament Supply/COMP_FB_FIL -> Net-(U6-REF)
- R53 pad 1: /Filament Supply/GATE_FIL -> Net-(R47-Pad2)
- R53 pad 2: Net-(Q3-G) -> Net-(D27-A)
- R54 pad 1: Net-(R50-Pad2) -> /Filament Supply/FILAMENT
- R54 pad 2: Net-(U6-K) -> Net-(D29-A)
- R55 pad 1: Net-(C37-Pad2) -> Net-(C51-Pad2)
- R55 pad 2: Net-(U6-REF) -> Net-(U7-REF)
- R56 pad 1: /Filament Supply/CS_FIL -> /Filament Supply/COMP_FB_FIL
- R56 pad 2: /Filament Supply/MOS_SOURCE_FIL -> Net-(C53-Pad1)
- R57 pad 1: /Filament Supply/COMP_FB_FIL -> Net-(U5-RT)
- R57 pad 2: Net-(C40-Pad1) -> AGND2
- R58 pad 1: /Filament Supply/VCC_FIL -> Net-(U6-REF)
- R58 pad 2: Net-(D18-A) -> /Filament Supply/CATHODE
- R59 pad 1: Net-(U6-REF) -> Net-(U7-REF)
- R6 pad 1: Net-(D5-A) -> /A3 Supply/CS_FILT
- R6 pad 2: Net-(D6-K) -> /A3 Supply/CS
- R60 pad 1: Net-(U5-RT) -> /Filament Supply/+12V_IN
- R60 pad 2: AGND2 -> Net-(D30-A)
- R7 pad 1: Net-(U1-GATE) -> /A3 Supply/VCC
- R7 pad 2: Net-(Q1-G) -> /A3 Supply/PGOOD_HV
- R8 pad 1: /A2 Supply/CS_FILT -> GND
- R8 pad 2: /A2 Supply/CS -> /A3 Supply/FB_PDA
- R9 pad 1: /A3 Supply/FB_PDA -> Net-(R9-Pad1)
- RS1 pad 1: /A2 Supply/CS -> /A3 Supply/CS
- RS2 pad 1: /A3 Supply/CS -> /A2 Supply/CS
- RV1 pad 1: /A2 Supply/-2KV -> /A3 Supply/FB_PDA
- RV1 pad 2: /A2 Supply/CATHODE -> /A3 Supply/FB_PDA
- RV1 pad 3: /A2 Supply/BRIGHTNESS -> Net-(R9-Pad1)
- RV2 pad 1: Net-(R15-Pad2) -> Net-(R25-Pad2)
- RV2 pad 2: Net-(R15-Pad2) -> Net-(R25-Pad2)
- RV3 pad 1: Net-(R46-Pad2) -> Net-(R59-Pad2)
- RV3 pad 2: /A3 Supply/FB_PDA -> /Filament Supply/CATHODE
- RV3 pad 3: /A3 Supply/FB_PDA -> /Filament Supply/CATHODE
- T1 pad 1: /A2 Supply/+12V_IN -> /A3 Supply/PDA_SEC
- T1 pad 2: /A2 Supply/+12V_IN -> unconnected-(T1-Pad2)
- T1 pad 3: /A2 Supply/MOS_DRAIN -> /A3 Supply/+12V_IN
- T1 pad 4: /A2 Supply/MOS_DRAIN -> /A3 Supply/+12V_IN
- T1 pad 5: GND -> /A3 Supply/+12V_IN
- T1 pad 6: (no net) -> /A3 Supply/+12V_IN
- T1 pad 7: (no net) -> /A3 Supply/MOS_DRAIN
- T1 pad 8: Net-(D2-K) -> /A3 Supply/MOS_DRAIN
- T2 pad 1: /A3 Supply/+12V_IN -> GND
- T2 pad 2: /A3 Supply/+12V_IN -> unconnected-(T2-Pad2)
- T2 pad 3: /A3 Supply/MOS_DRAIN -> /A2 Supply/+12V_IN
- T2 pad 4: /A3 Supply/MOS_DRAIN -> /A2 Supply/+12V_IN
- T2 pad 5: Net-(D13-A) -> /A2 Supply/+12V_IN
- T2 pad 6: (no net) -> /A2 Supply/+12V_IN
- T2 pad 7: (no net) -> /A2 Supply/MOS_DRAIN
- T2 pad 8: GND -> /A2 Supply/MOS_DRAIN
- T3 pad 7: Net-(D17-A) -> Net-(D25-A)
- T3 pad 8: Net-(D17-A) -> Net-(D25-A)
- U1 pad 1: /A2 Supply/+12V_IN -> /A3 Supply/+12V_IN
- U1 pad 11: /A2 Supply/PGOOD_HV -> /A3 Supply/PGOOD_HV
- U1 pad 12: /A2 Supply/UVLO -> /A3 Supply/UVLO
- U1 pad 2: /A2 Supply/VCC -> /A3 Supply/VCC
- U1 pad 5: /A2 Supply/CS_FILT -> /A3 Supply/CS_FILT
- U1 pad 7: AGND -> AGND3
- U1 pad 8: /A2 Supply/FB_HV -> /A3 Supply/FB_PDA
- U2 pad 1: /A2 Supply/FB_HV -> /A2 Supply/+12V_IN
- U2 pad 2: GND -> /A2 Supply/VCC
- U2 pad 3: GND -> Net-(U2-GATE)
- U2 pad 4: /A2 Supply/FB_HV_LADDER -> GND
- U2 pad 5: /A2 Supply/VCC -> /A2 Supply/CS_FILT
- U3 pad 1: /A3 Supply/+12V_IN -> /A2 Supply/FB_HV
- U3 pad 2: /A3 Supply/VCC -> GND
- U3 pad 3: Net-(U3-GATE) -> GND
- U3 pad 4: GND -> /A2 Supply/FB_HV_LADDER
- U3 pad 5: /A3 Supply/CS_FILT -> /A2 Supply/VCC
- U4 pad 1: Net-(R50-Pad2) -> Net-(R47-Pad2)
- U4 pad 2: Net-(U6-K) -> Net-(D27-A)
- U5 pad 11: /Filament Supply/PGOOD_FIL -> unconnected-(U5-PGOOD-Pad11)
- U5 pad 3: /Filament Supply/GATE_FIL -> Net-(U5-GATE)
- U6 pad 1: Net-(U6-K) -> /Filament Supply/TRIAC_GATE
Routing:
- net (no net): track 335.9 -> 0.00 mm, vias 7 -> 0
- net /Filament Supply/+12V_IN: track 77.4 -> 165.8 mm, vias 4 -> 1
- net /A2 Supply/+12V_IN: track 59.1 -> 144.3 mm, vias 2 -> 4
- net /Filament Supply/CATHODE: track 85.0 -> 165.2 mm
- net /A2 Supply/PGOOD_HV: track 18.5 -> 93.7 mm
- net /A2 Supply/-2KV: track 74.0 -> 0.00 mm
- net /A3 Supply/FB_PDA: track 76.3 -> 19.5 mm
- net /Filament Supply/UNFUSED_FILAMENT: track 0.00 -> 55.7 mm, vias 0 -> 2
- net /A3 Supply/+12V_IN: track 57.5 -> 110.2 mm
- net /A2 Supply/CATHODE: track 49.1 -> 0.00 mm
- net Net-(U6-K): track 47.7 -> 0.00 mm
- net Net-(R9-Pad1): track 0.00 -> 38.1 mm, vias 0 -> 2
- net /A2 Supply/-HV: track 0.00 -> 36.6 mm
- net /Filament Supply/FILAMENT: track 124.0 -> 89.7 mm, vias 0 -> 1
- net GND: track 176.2 -> 142.6 mm, vias 60 -> 25
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- added copper zone on F.Cu, net /A2 Supply/MOS_DRAIN
- added copper zone on F.Cu, net /A3 Supply/MOS_DRAIN
- removed copper zone on F.Cu, net /A2 Supply/CATHODE
Other:
- outline, holes or cut-outs redrawn
- board text added: "+"
- board text added: "+12V GND"
- board text added: "+400 to +2000V A3 -400 to -2000V A2 6.3V PROTECTED HEATER"
- board text added: "-"
- board text added: "6.3V ONLY NO 2.5V FILAMENTS GO HOME 3AP/5MP"
- board text added: "6.6V OVP CROWBAR WILL BLOW FUSE"
- board text added: "9/10 toothpaste brands approve of this dentist"
- board text added: "A2 EN"
- board text added: "A2 ENABLE"
- board text added: "A2 OK"
- board text added: "A3"
- board text added: "A3 EN"
- board text added: "A3 ENABLE"
- board text added: "A3 OK"
- board text added: "ADJUST HEATER 5.7 - 6.4V"
- board text added: "CATHODE"
- board text added: "CRT HIGH VOLTAGE SUPPLY V3.5"
- board text added: "CSD FETS from TI stand for CURRENT SENSITIVE DISGRACE"
- board text added: "CSD19873 FET GRAVEYARD, COLMA, CA"
- board text added: "FET"
- board text added: "H+ H-"
- board text added: "HEATER ENABLE"
- board text added: "HEATER OK"
- board text added: "IF YOU REMOVED THIS PART THEN COILCRAFT LIED ABOUT THE 1500V RMS HI-POT RATING AND YOU SHOULD BULLY THEM FOR IT"
- board text added: "LIKE A G6? WHAT KIND OF TUBE DO YOU HAVE THAT HAS 6 GRIDS???"
- board text added: "NON-MONETARY COMPENSATION"
- board text added: "STATUS BAR (drinks served after 9PM)"
- board text added: "chibitron.com"
- board text added: "cockroft walton multiplier ha...he said COCK"
- board text added: "do not sue me if you touch here"
- board text added: "please refrain from climbing resistor ladder"
- board text added: "this circuit is basically the cha-cha slide for electrons"
- board text removed: "0-50% of A2 (Now isolated for your protection)"
- board text removed: "BOURNS Y U NO MAKE 1000V POTENTIOMETER"
- board text removed: "COSTCO"
- board text removed: "CRT Main Supply 3 2KV x2 + 6.3V"
- board text removed: "FOCUS"
- board text removed: "I applied 12V to this circuit and all I got was this lit-up LED"
- board text removed: "Packing Peanut"
- board text removed: "chibi"
- board text removed: "do not eat the coilcraft sample transformer"
- board text removed: "don't touch i bite :3"
- board text removed: "this is not a fucking"
- board text removed: "{DMZ} DO NOT CROSS"
