File: main_supply_3_revised/main_supply_3_revised/main_supply_3_revised.kicad_sch (KiCad schematic)
At the start: 9 parts, among them J1 Conn_01x02_Pin, J10 12V PASS, J11 FILAMENT, J12 GRID, J2 A3_EN, J3 Conn_01x05, J5 A2_EN, J6 FIL_EN

Commit message: defl 5 + mainboard 3
Parts:
- removed J12: GRID, symbol Connector_Generic:Conn_01x02
- removed J3: Conn_01x05, symbol Connector_Generic:Conn_01x05
- added J4: HV OUT, Connector_JST:JST_VH_B5P-VH-B_1x05_P3.96mm_Vertical, symbol Connector_Generic:Conn_01x05_3P_SP
- F1: footprint Fuse:Fuse_0805_2012Metric -> Fuse:Fuseholder_Littelfuse_Nano2_154x
- J6: renamed from J11; footprint (none) -> Connector_JST:JST_VH_B2P-VH-B_1x02_P3.96mm_Vertical
- renumbered J10 to J2, J2 to J3, J6 to J7
Connections:
- net +12V: now also J2.1 (Pin_1)
- net A3 Supply/+PDA: now also J4.1 (Pin_1)
- net GND: now also J2.2 (Pin_2), J4.3 (Pin_3)
- new net A2 Supply/-HV: J4.5 (Pin_5)
Other:
- sheet A2 Supply ports: added -HV; removed -2KV, CATHODE
- moved on the sheet: F1, J1
