File: main_supply_4_VM/_autosave-main_supply_4_VM.kicad_pcb (KiCad board)
At the start: 2 copper layers, 100 x 100 mm, 187 parts, among them J1 Conn_01x02_Pin, J2 A3_EN, J3 12V_PASS, J4 MAIN_HV, J5 A2_EN, J6 FIL_EN, J7 FILAMENT, Q1 2N7002, Q2 Si7450DP, Q3 2N7002, Q4 Si7450DP, Q5 2N7002, Q6 Si7450DP, T1 750315839, T2 750315839, T3 YA9033-ALD, U1 AP2204K-5.0, U2 LM5155DSSR, U3 TLV314QDBVR, U4 LM5155DSSR, U5 TLV314QDBVR, U6 TLV314QDBVR, U7 PC817, U8 LM5155DSSR, U9 TL431DBZ

Commit message: finished routing and layout
need to update U6 stuff
Parts:
- removed the J3 at (55.3, 4.18)
- removed the J4 at (26.1, 96.8)
- added C51: 10n, Capacitor_SMD:C_2220_5750Metric, F.Cu at (192.8, 75.2)
- added C52: 10n, Capacitor_SMD:C_2220_5750Metric, F.Cu at (192.8, 106.4)
- added J5: MAIN HV, JST_VH:JST_VH_B3P5-VH-B_1x05_P3.96mm_Vertical, F.Cu at (195.2, 83.0)
- added R84: 1.5k, Resistor_SMD:R_1206_3216Metric, F.Cu at (193.6, 68.2)
- added R85: 1.5k, Resistor_SMD:R_1206_3216Metric, F.Cu at (192.6, 115.0)
- added TP3: AGND3, TestPoint:TestPoint_Keystone_5010-5014_Multipurpose, F.Cu at (120.0, 83.2)
- added TP4: AGND, TestPoint:TestPoint_Keystone_5010-5014_Multipurpose, F.Cu at (120.0, 116.8)
- added TP5: 5V, TestPoint:TestPoint_Keystone_5010-5014_Multipurpose, F.Cu at (110.2, 141.0)
- J1: value Conn_01x02_Pin -> 12V IN; footprint Connector_Molex:Molex_KK-396_5273-02A_1x02_P3.96mm_Vertical -> Connector_JST:JST_VH_B2P-VH-B_1x02_P3.96mm_Vertical
- NT1, NT2, NT3: footprint NetTie:NetTie-2_SMD_Pad0.5mm -> NetTie:NetTie_0.2mm
- R12: value 22k -> 39k
- RV1, RV2: footprint Potentiometer_THT:Potentiometer_Bourns_3296W_Vertical -> Potentiometer_THT:Potentiometer_Bourns_3296Y_Vertical
- U2, U4, U8: footprint LM5155:IC_LM5155DSSR -> LM5155DSSR:IC_LM5155DSSR
- moved Q6 187.0 mm to (136.6, 136.2)
- moved J6 185.7 mm to (195.2, 137.2), turned to -90 degrees
- moved C27 171.1 mm to (181.7, 93.6)
- moved R1 169.7 mm to (194.2, 122.6), turned to -90 degrees
- moved C25 163.7 mm to (173.4, 93.6)
- moved R2 161.4 mm to (178.8, 67.5)
- moved D13 158.7 mm to (182.8, 105.7), turned to 90 degrees
- moved C23 156.5 mm to (165.1, 93.6)
- moved D12 155.1 mm to (178.2, 105.7), turned to -90 degrees
- moved D1 155.0 mm to (186.3, 62.3), turned to 90 degrees
- moved R44 153.7 mm to (183.4, 99.4)
- moved D11 151.6 mm to (173.8, 105.7), turned to 90 degrees
- moved R6 150.7 mm to (168.6, 67.5)
- moved T1 150.0 mm to (150.0, 62.0), turned to 90 degrees
- moved C45 149.5 mm to (176.0, 134.8), turned to -90 degrees
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- renumbered J5 to J3, J6 to J4, J7 to J6, R27 to R15, R28 to R16, R29 to R17, R30 to R18, R31 to R19, R32 to R20, R33 to R21, R34 to R22, R99 to R23, R100 to R24, R101 to R25, R102 to R26, R103 to R27, R92 to R28, R89 to R29, R86 to R30, R104 to R31, R105 to R32, R106 to R33, R107 to R34, R61 to R49, R62 to R50, R63 to R51, R64 to R52, R65 to R53, R98 to R54, R97 to R55, R96 to R56, R95 to R57, R94 to R58, R91 to R59, R88 to R60, R85 to R61, R93 to R62, R90 to R63, R87 to R64, R84 to R65
Connections:
- net /A3 Supply/+PDA renamed /A3 Supply/PDA_FB
- net Net-(Q2-D) renamed /A3 Supply/GATE_DRAIN
- net Net-(Q4-D) renamed /A2 Supply/GATE_DRAIN
- C27 pad 2: /A2 Supply/-2KV -> /A2 Supply/A2_FB
- F1 pad 1: Net-(J1-Pin_1) -> /12V_IN
- J1 pad 1: Net-(J1-Pin_1) -> GND
- J1 pad 2: GND -> /12V_IN
- Q5 pad 2: AGND -> AGND2
- R1 pad 2: /Filament Supply/FILAMENT -> /Filament Supply/CATHODE
- R12 pad 1: /A3 Supply/VCC -> +12V
- R18 pad 2: Net-(R30-Pad2) -> Net-(R18-Pad2)
- R21 pad 1: Net-(R33-Pad1) (its old number) -> Net-(R21-Pad1)
- R44 pad 2: /A2 Supply/-2KV -> /A2 Supply/A2_FB
- R46 pad 1: /A2 Supply/VCC -> +12V
- R50 pad 2: Net-(R62-Pad2) -> Net-(R50-Pad2)
- R53 pad 1: Net-(R65-Pad1) -> Net-(R53-Pad1)
- R65 pad 1: /A2 Supply/-2KV -> /A2 Supply/A2_FB
- R70 pad 2: AGND -> AGND2
- RV1 pad 1: Net-(R30-Pad2) -> Net-(R21-Pad1)
- RV1 pad 3: Net-(R33-Pad1) (its old number) -> Net-(R18-Pad2)
- RV2 pad 1: Net-(R62-Pad2) -> Net-(R53-Pad1)
- RV2 pad 3: Net-(R65-Pad1) -> Net-(R50-Pad2)
- RV3 pad 1: Net-(R83-Pad2) -> /Filament Supply/CATHODE
- RV3 pad 3: /Filament Supply/CATHODE -> Net-(R83-Pad2)
- U8 pad 8: GND -> AGND2
Routing:
- net +5V: track 0.00 -> 160.0 mm, vias 0 -> 7
- net +12V: track 0.00 -> 97.5 mm, vias 0 -> 68
- net /Filament Supply/CATHODE: track 0.00 -> 96.1 mm, vias 0 -> 2
- net GND: track 0.00 -> 85.5 mm, vias 0 -> 60
- net /A2 Supply/EN: track 0.00 -> 53.2 mm, vias 0 -> 1
- net /A3 Supply/EN: track 0.00 -> 52.1 mm, vias 0 -> 1
- net /Filament Supply/EN: track 0.00 -> 49.1 mm
- net /Filament Supply/FILAMENT: track 0.00 -> 47.3 mm, vias 0 -> 2
- net Net-(C18-Pad1): track 0.00 -> 39.3 mm, vias 0 -> 1
- net /A2 Supply/A2_FB: track 0.00 -> 30.7 mm
- net Net-(U6-+): track 0.00 -> 29.7 mm, vias 0 -> 1
- net Net-(D18-A): track 0.00 -> 26.7 mm
- net /A3 Supply/PDA_FB: track 0.00 -> 23.7 mm
- net /A2 Supply/-2KV: track 0.00 -> 22.6 mm
- net /Filament Supply/COMP_FB_FIL: track 0.00 -> 21.2 mm, vias 0 -> 3
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- added copper zone on B.Cu, net +12V
- added copper zone on F.Cu, net +12V
- added copper zone on F.Cu, net /12V_IN
- added copper zone on F.Cu, net /A2 Supply/GATE_DRAIN
- added copper zone on F.Cu, net /A3 Supply/GATE_DRAIN
- added copper zone on F.Cu, net /Filament Supply/FILAMENT
- added copper zone on F.Cu, net /Filament Supply/MOS_DRAIN_FIL
- added copper zone on F.Cu, net /Filament Supply/MOS_SOURCE_FIL
- added copper zone on F.Cu, net AGND
- added copper zone on F.Cu, net AGND2
- added copper zone on F.Cu, net AGND3
- added copper zone on B.Cu, net GND
- added copper zone on F.Cu, net GND
Other:
- outline, holes or cut-outs redrawn
- board text added: "+"
- board text added: "+12V GND"
- board text added: "+5V"
- board text added: "-"
- board text added: "400V 2KV"
- board text added: "400V-2KV x2 6.3V FILAMENT"
- board text added: "5.7V-6.4V"
- board text added: "A1"
- board text added: "A2"
- board text added: "A2 EN A2 OK"
- board text added: "A3"
- board text added: "A3 EN A3 OK"
- board text added: "AGND"
- board text added: "CRT High Voltage Supply V.4"
- board text added: "CRT Phosphor Types: Code: Flourescent color, Persistence time (phosphorescent color) P1: Green, Medium P2: Green, Medium-Long - P4: White, Medium-Short P5: Blue, Medium-Short - P7: Whitish-Blue, Long (Yellow) - P10: Reflective Pink, Long (non-emissive) P11: Actinic Blue, Medium-Short P12: Amber, Medium-Long - P15: Blue-Green, Very-short P16: Violet/UV-A, Very-short - P19: Amber, Long - P22: R,G,B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"
- board text added: "D3"
- board text added: "D4"
- board text added: "DISABLE HV BEFORE ADJUSTMENT"
- board text added: "DO NOT TOUCH OUTPUT"
- board text added: "ENABLE A2"
- board text added: "ENABLE A3"
- board text added: "ENABLE HEATER"
- board text added: "FIL ON"
- board text added: "G1"
- board text added: "H"
- board text added: "H+"
- board text added: "H-"
- board text added: "HEATER"
- board text added: "HV MAIN"
- board text added: "Just remember: ChatGPT said this project was too dangerous for me to make. I did it anyway."
- board text added: "K"
- board text added: "MEASURE A2 HERE (1:1000)"
- board text added: "MEASURE A3 HERE (1:1000)"
- board text added: "PLUG DDR5 INTO HV MAIN"
- board text added: "This board generates: H A2 A3 Deflection board generates: A1 from A2 D1 - D4 G1"
- board text added: "UP TO 4KV PRESENT"
- board text added: "chibitron.com"
- board text added: "do not aim beam at eyes"
- board text added: "viagra is not a soft-start but two diodes & an RC filter is."
- board text added: "why did you put an indicator LED here? This circuit literally powers a lightbulb."
