File: main_supply_4_VM/hv_pos.kicad_sch (KiCad schematic)
At the start: 52 parts, among them Q1 2N7002, Q2 Si7450DP, T1 750315839, U2 LM5155DSSR, U3 TLV314QDBVR

Commit message: finished routing and layout
need to update U6 stuff
Parts:
- added C51: 10n, Capacitor_SMD:C_2220_5750Metric, symbol Device:C
- added R84: 1.5k, Resistor_SMD:R_1206_3216Metric, symbol Device:R_US
- added TP3: AGND3, TestPoint:TestPoint_Keystone_5010-5014_Multipurpose, symbol Connector:TestPoint
- NT1: footprint NetTie:NetTie-2_SMD_Pad0.5mm -> NetTie:NetTie_0.2mm
- R12: value 22k -> 39k
- R15: renamed from R27; value R_US -> 12k
- R18: renamed from R30; value 30k -> 18.7k
- R20: renamed from R32; value R_US -> 3k
- R21: renamed from R33; value 2.4k -> 2.49k
- R7: value 10k -> 1k
- RV1: footprint Potentiometer_THT:Potentiometer_Bourns_3296W_Vertical -> Potentiometer_THT:Potentiometer_Bourns_3296Y_Vertical
- U2: footprint LM5155:IC_LM5155DSSR -> LM5155DSSR:IC_LM5155DSSR
- renumbered R28 to R16, R29 to R17, R31 to R19, R34 to R22
Connections:
- net +12V_IN: now also R12.1
- net +PDA: now also C51.1, R84.2; no longer C5.2, D1.1 (K)
- net AGND3: now also TP3.1
- net GND: now also C51.2
- net VCC: no longer R12.1
- net at RV1.1: now also R21.1; no longer R18.2
- net at RV1.3: now also R18.2; no longer R21.1
- net GATE_DRAIN: now reaches Q2.5 (D), R9.2, T1.3
- new net PDA_FB: C5.2, D1.1 (K), R84.1
Other:
- note added: "basically U3 creates a buffered voltage, being subtracted as 2-(TP1) TP1 (A3-ADJ) should represent output voltage at scale 1000:1"
- moved on the sheet: C10, C11, C12, C13, C14, C15, C16, C17, C18, C19, C4, C5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
