File: main_supply_4_VM/main_supply_4_VM.kicad_sch (KiCad schematic)
At the start: 13 parts, among them J1 Conn_01x02_Pin, J2 A3_EN, J3 12V_PASS, J4 MAIN_HV, J5 A2_EN, J6 FIL_EN, J7 FILAMENT, U1 AP2204K-5.0

Commit message: finished routing and layout
need to update U6 stuff
Parts:
- removed J1: Conn_01x02_Pin, Connector_Molex:Molex_KK-396_5273-02A_1x02_P3.96mm_Vertical, symbol Connector:Conn_01x02_Pin
- removed J3: 12V_PASS, Connector_JST:JST_VH_B2P-VH-B_1x02_P3.96mm_Vertical, symbol Connector_Generic:Conn_01x02
- removed J4: MAIN_HV, Connector_JST:JST_VH_B5P-VH-B_1x05_P3.96mm_Vertical, symbol Connector_Generic:Conn_01x05_3P_SP
- added J1: 12V IN, Connector_JST:JST_VH_B2P-VH-B_1x02_P3.96mm_Vertical, symbol Connector_Generic:Conn_01x02
- added J5: MAIN HV, JST_VH:JST_VH_B3P5-VH-B_1x05_P3.96mm_Vertical, symbol JST-VH:Conn_01x03x05
- added TP5: 5V, TestPoint:TestPoint_Keystone_5010-5014_Multipurpose, symbol Connector:TestPoint
- renumbered J5 to J3, J6 to J4, J7 to J6
Connections:
- net +5V: now also TP5.1
- net A2 Supply/-2KV: now also J5.5 (Pin_5)
- net A3 Supply/+PDA: now also J5.1 (Pin_1)
- net Filament Supply/CATHODE: now also R1.2
- net Filament Supply/FILAMENT: no longer R1.2
- net GND: now also J1.1 (Pin_1), J5.3 (Pin_3)
- net 12V_IN: now reaches F1.1
- net 12V_IN: now also J1.2 (Pin_2)
