File: main_supply_4_VM/filament.kicad_sch (KiCad schematic)
At the start: 46 parts, among them Q5 2N7002, Q6 Si7450DP, T3 YA9033-ALD, U7 PC817, U8 LM5155DSSR, U9 TL431DBZ

Commit message: testload
Parts:
- C45: value C -> 4.7u
- R72: value R_US -> 100k
Other:
- moved on the sheet: D17, D18
Changed lines of the file:
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@@
 	(text "secondary\nside\nsoft-start"
 		(exclude_from_sim no)
-		(at 293.37 87.122 0)
+		(at 292.608 87.122 0)
 		(effects
 			(font
@@
 	)
 	(junction
-		(at 289.56 92.71)
+		(at 288.29 92.71)
 		(diameter 0)
 		(color 0 0 0 0)
@@
 	)
 	(junction
-		(at 289.56 135.89)
+		(at 288.29 135.89)
 		(diameter 0)
 		(color 0 0 0 0)
@@
 	)
 	(junction
-		(at 289.56 110.49)
+		(at 288.29 110.49)
 		(diameter 0)
 		(color 0 0 0 0)
@@
 	(wire
 		(pts
-			(xy 289.56 92.71) (xy 289.56 101.6)
+			(xy 288.29 92.71) (xy 288.29 101.6)
 		)
 		(stroke
@@
 	(wire
 		(pts
-			(xy 278.13 92.71) (xy 289.56 92.71)
+			(xy 278.13 92.71) (xy 288.29 92.71)
 		)
 		(stroke
@@
 	(wire
 		(pts
-			(xy 289.56 110.49) (xy 297.18 110.49)
+			(xy 288.29 110.49) (xy 297.18 110.49)
 		)
 		(stroke
@@
 	(wire
 		(pts
-			(xy 278.13 135.89) (xy 289.56 135.89)
+			(xy 278.13 135.89) (xy 288.29 135.89)
 		)
 		(stroke
@@
 	(wire
 		(pts
-			(xy 289.56 92.71) (xy 297.18 92.71)
+			(xy 288.29 92.71) (xy 297.18 92.71)
 		)
 		(stroke
@@
 	(polyline
 		(pts
-			(xy 288.29 91.44) (xy 288.29 90.17)
+			(xy 287.02 91.44) (xy 287.02 90.17)
 		)
 		(stroke
@@
 	(wire
 		(pts
-			(xy 289.56 109.22) (xy 289.56 110.49)
+			(xy 288.29 109.22) (xy 288.29 110.49)
 		)
 		(stroke
@@
 	(wire
 		(pts
-			(xy 289.56 119.38) (xy 289.56 135.89)
+			(xy 288.29 119.38) (xy 288.29 135.89)
 		)
 		(stroke
@@
 	(polyline
 		(pts
-			(xy 288.29 90.17) (xy 298.45 90.17)
+			(xy 287.02 90.17) (xy 298.45 90.17)
 		)
 		(stroke
@@
 	(wire
 		(pts
-			(xy 289.56 135.89) (xy 292.1 135.89)
+			(xy 288.29 135.89) (xy 292.1 135.89)
 		)
 		(stroke
@@
 	(wire
 		(pts
-			(xy 289.56 110.49) (xy 289.56 111.76)
+			(xy 288.29 110.49) (xy 288.29 111.76)
 		)
 		(stroke
@@
 	(symbol
 		(lib_id "Device:D_Schottky")
-		(at 289.56 105.41 270)
+		(at 288.29 105.41 270)
 		(unit 1)
 		(exclude_from_sim no)
@@
 		(fields_autoplaced yes)
 		(property "Reference" "D17"
-			(at 292.1 105.0924 90)
+			(at 290.83 105.0924 90)
 			(effects
 				(font
@@
 		)
 		(property "Value" "D_Schottky"
-			(at 292.1 106.3624 90)
+			(at 290.83 106.3624 90)
 			(effects
 				(font
@@
 		)
 		(property "Footprint" "Diode_SMD:D_SOD-123"
-			(at 289.56 105.41 0)
+			(at 288.29 105.41 0)
 			(effects
 				(font
@@
 		)
 		(property "Datasheet" "~"
-			(at 289.56 105.41 0)
+			(at 288.29 105.41 0)
 			(effects
 				(font
@@
 		)
 		(property "Description" "Schottky diode"
-			(at 289.56 105.41 0)
+			(at 288.29 105.41 0)
 			(effects
 				(font
@@
 		)
 		(property "Sim.Type" ""
-			(at 289.56 105.41 0)
+			(at 288.29 105.41 0)
 			(effects
 				(font
@@
 	(symbol
 		(lib_id "Device:D_Schottky")
-		(at 289.56 115.57 270)
+		(at 288.29 115.57 270)
 		(unit 1)
 		(exclude_from_sim no)
@@
 		(fields_autoplaced yes)
 		(property "Reference" "D18"
-			(at 292.1 115.2524 90)
+			(at 290.83 115.2524 90)
 			(effects
 				(font
@@
 		)
 		(property "Value" "D_Schottky"
-			(at 292.1 116.5224 90)
+			(at 290.83 116.5224 90)
 			(effects
 				(font
@@
 		)
 		(property "Footprint" "Diode_SMD:D_SOD-123"
-			(at 289.56 115.57 0)
+			(at 288.29 115.57 0)
 			(effects
 				(font
@@
 		)
 		(property "Datasheet" "~"
-			(at 289.56 115.57 0)
+			(at 288.29 115.57 0)
 			(effects
 				(font
@@
 		)
 		(property "Description" "Schottky diode"
-			(at 289.56 115.57 0)
+			(at 288.29 115.57 0)
 			(effects
 				(font
@@
 		)
 		(property "Sim.Type" ""
-			(at 289.56 115.57 0)
+			(at 288.29 115.57 0)
 			(effects
 				(font
@@
 			)
 		)
-		(property "Value" "C"
+		(property "Value" "4.7u"
 			(at 300.99 118.1099 0)
 			(effects
@@
 			)
 		)
-		(property "Value" "R_US"
+		(property "Value" "100k"
 			(at 299.72 105.4099 0)
 			(effects
